Commit message: Changed settings in URDF

File: ros2_control_demo_description/diffbot_description/ros2_control/diffbot.ros2_control.xacro (robot description, xacro)
@@ -5,5 +5,5 @@
       <hardware>
         <plugin>ros2_control_demo_hardware/DiffBotSystemHardware</plugin>
-        <param name="example_param_hw_start_duration_sec">0</param>
+        <param name="example_param_hw_start_duration_sec">0.5</param>
         <param name="example_param_hw_stop_duration_sec">3.0</param>
       </hardware>

File: ros2_control_demo_description/diffbot_description/urdf/diffbot_description.urdf.xacro (robot description, xacro)
@@ -5,12 +5,12 @@
   <xacro:property name="PI" value="3.1415926535897931"/>
   <xacro:property name="base_mass" value="0.3" /> <!-- arbitrary value for base mass -->
-  <xacro:property name="base_width" value="0.1" />
-  <xacro:property name="base_length" value="0.1" />
+  <xacro:property name="base_width" value="0.3" />
+  <xacro:property name="base_length" value="0.3" />
   <xacro:property name="base_height" value="0.05" />
   <xacro:property name="wheel_mass" value="0.3" /> <!-- arbitrary value for wheel mass -->
   <xacro:property name="wheel_len" value="0.020" />
-  <xacro:property name="wheel_radius" value="0.015" />
+  <xacro:property name="wheel_radius" value="0.060" />
   <xacro:property name="caster_wheel_mass" value="0.1" /> <!-- arbitrary value for caster wheel mass -->
-  <xacro:property name="caster_wheel_radius" value="0.015" />
+  <xacro:property name="caster_wheel_radius" value="0.045" />
   <xacro:property name="z_offset" value="-${base_height/2}" /> <!-- Space btw top of beam and the each joint -->
   <!-- Base Link -->
@@ -29,4 +29,12 @@
       <material name="orange"/>
     </visual>
+    <inertial>
+      <origin xyz="0 0 0" rpy="0 0 0"/>
+      <mass value="${base_mass}"/>
+      <inertia
+        ixx="${base_mass / 12.0 * (base_length*base_length + base_height*base_height)}" ixy="0.0" ixz="0.0"
+        iyy="${base_mass / 12.0 * (base_height*base_height + base_width*base_width)}" iyz="0.0"
+        izz="${base_mass / 12.0 * (base_width*base_width + base_length*base_length)}"/>
+    </inertial>
     </link>
     <joint name="${prefix}left_wheel_joint" type="continuous">
