Commit message: Removed inertial param from base link to play nicely

File: ros2_control_demo_description/diffbot_description/urdf/diffbot_description.urdf.xacro (robot description, xacro)
@@ -29,12 +29,4 @@
       <material name="orange"/>
     </visual>
-    <inertial>
-      <origin xyz="0 0 0" rpy="0 0 0"/>
-      <mass value="${base_mass}"/>
-      <inertia
-        ixx="${base_mass / 12.0 * (base_length*base_length + base_height*base_height)}" ixy="0.0" ixz="0.0"
-        iyy="${base_mass / 12.0 * (base_height*base_height + base_width*base_width)}" iyz="0.0"
-        izz="${base_mass / 12.0 * (base_width*base_width + base_length*base_length)}"/>
-      </inertial>
     </link>
     <joint name="${prefix}left_wheel_joint" type="continuous">
